Commit message: account for robotiq and umi fingers in tool0

File: fixed_unload_xarm7.urdf (robot description, URDF)
Before this commit: robot xarm7, 9 links, 8 joints
Joints:
- joint unload_left_link7-tool0_fixed_joint: origin xyz=0 0 0 rpy=0 0 -0.785398 -> xyz=0 0 0.0247 rpy=0 0 -1.5707963267948966
